File: ag-diy-pro.kicad_pcb (KiCad board)
At the start: 2 copper layers, 79.6 x 62.5 mm, 48 parts, among them U2 TPL5010, U3 SGP41-D-R4, U4 LM1117-3.3, U5 SHT4XI-DIGITAL, U6 ESP32-C3-MINI-1-N4

Commit message: first working draft and verified build
Other:
- outline, holes or cut-outs redrawn
Changed lines of the file:
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@@
 			(psa4output no)
 			(plot_black_and_white yes)
-			(plotinvisibletext no)
 			(sketchpadsonfab no)
 			(plotpadnumbers no)
@@
 		)
 		(property "Value" "SGP41-D-R4"
-			(at -0.3 1.88 0)
+			(at 4.421 2.0764 0)
 			(layer "F.Fab")
 			(effects
@@
 		(at 96.52 40.305)
 		(property "Reference" "U6"
-			(at 0 0 0)
+			(at -3.675 -9.635 0)
 			(layer "F.SilkS")
 			(effects
@@
 		)
 		(property "Value" "ESP32-C3-MINI-1-N4"
-			(at -0.02 9.395 0)
+			(at 7.755 9.635 0)
 			(layer "F.Fab")
 			(effects
@@
 		(descr "Industrial SHT4xI-DigitalDFN150X150X54-4N")
 		(property "Reference" "U5"
-			(at 1.7 0.038927 90)
+			(at 1.975 -1.635 0)
 			(layer "F.SilkS")
 			(effects
@@
 		)
 		(property "Value" "SHT4XI-DIGITAL"
-			(at -1.2 -4.561073 90)
-			(layer "B.Fab")
+			(at 7.59 1.665 0)
+			(layer "F.Fab")
 			(effects
 				(font
@@
 	)
 	(gr_line
-		(start 119.03 32.505)
+		(start 119.03 32.38)
 		(end 119.03 31.495)
 		(stroke
@@
 	)
 	(gr_line
-		(start 147.57 32.58)
-		(end 156.9 32.58)
+		(start 147.57 32.45)
+		(end 156.9 32.45)
 		(stroke
 			(width 0.2)
@@
 	)
 	(gr_line
-		(start 119.03 37.88)
-		(end 119.03 36.08)
+		(start 119.44 37.65)
+		(end 119.44 36.08)
 		(stroke
 			(width 0.2)
@@
 	)
 	(gr_line
-		(start 138.97 32.53)
+		(start 138.97 32.4)
 		(end 138.97 31.52)
 		(stroke
@@
 	)
 	(gr_line
-		(start 136.43 32.53)
-		(end 138.97 32.53)
+		(start 136.43 32.4)
+		(end 138.97 32.4)
 		(stroke
 			(width 0.2)
@@
 	(gr_line
 		(start 121.57 31.495)
-		(end 121.57 32.505)
+		(end 121.57 32.38)
 		(stroke
 			(width 0.2)
@@
 	)
 	(gr_line
-		(start 156.9 32.58)
+		(start 156.9 32.45)
 		(end 156.9 31.538)
 		(stroke
@@
 	(gr_line
 		(start 147.57 31.53)
-		(end 147.57 32.58)
+		(end 147.57 32.45)
 		(stroke
 			(width 0.2)
@@
 	)
 	(gr_line
-		(start 121.57 32.505)
-		(end 119.03 32.505)
+		(start 121.57 32.38)
+		(end 119.03 32.38)
 		(stroke
 			(width 0.2)
@@
 	(gr_line
 		(start 136.43 31.54)
-		(end 136.43 32.53)
+		(end 136.43 32.4)
 		(stroke
 			(width 0.2)
@@
 	)
 	(gr_line
-		(start 119.03 36.08)
+		(start 119.44 36.08)
 		(end 121.57 36.08)
 		(stroke
@@
 	(gr_line
 		(start 121.57 36.08)
-		(end 121.57 37.88)
+		(end 121.57 37.65)
 		(stroke
 			(width 0.2)
@@
 	)
 	(gr_line
-		(start 121.57 37.88)
-		(end 119.03 37.88)
+		(start 121.57 37.65)
+		(end 119.44 37.65)
 		(stroke
 			(width 0.2)
