File: ag-diy-pro.kicad_sch (KiCad schematic)
At the start: 43 parts, among them U2 TPL5010, U3 SGP41-D-R4, U4 LM1117-3.3, U5 SHT4XI-DIGITAL, U6 ESP32-C3-MINI-1-N4

Commit message: first working draft and verified build
Parts:
- Boot1, Reset1: LCSC Part # (none) -> C221855
- C1, C9: LCSC Part # (none) -> C1589
- C10, C12, C13, C17, C18, C19, C2, C3, C4, C6, C8: LCSC Part # (none) -> C1590
- C11, C16: LCSC Part # (none) -> C86295
- C20, C21: LCSC Part # (none) -> C5673
- C7: LCSC Part # (none) -> C96446
- F1: LCSC Part # (none) -> C70075
- IO1, PM2: LCSC Part # (none) -> C240845
- R10, R11: LCSC Part # (none) -> C25804
- R15: LCSC Part # (none) -> C23164
- R16, R17: LCSC Part # (none) -> C166926
- R4, R8: LCSC Part # (none) -> C25803
- R5: LCSC Part # (none) -> C23196
- R6, R7: LCSC Part # (none) -> C23186
- U2: LCSC Part # (none) -> C473912
- U3: LCSC Part # (none) -> C3659325
- U4: LCSC Part # (none) -> C6186
- U5: LCSC Part # (none) -> C9900186997
- U6: LCSC Part # (none) -> C2934561
- USB1: LCSC Part # (none) -> C168704
