File: ag-diy-pro.kicad_sch (KiCad schematic)
At the start: 43 parts, among them U2 TPL5010, U3 SGP41-D-R4, U4 LM1117-3.3, U5 SHT4XI-DIGITAL, U6 ESP32-C3-MINI-1-N4

Commit message: Revised
Parts:
- removed C10, C12, C2, C8: 0.1uf, Capacitor_SMD:C_0603_1608Metric, symbol Device:C
- removed C11: 22uf / 10V, Capacitor_SMD:C_0603_1608Metric, symbol Device:C
- removed C7: 10uf / 25V, Capacitor_SMD:C_0603_1608Metric, symbol Device:C
- removed I2C1, I2C2, I2C3: Conn_01x04, Connector_PinSocket_2.54mm:PinSocket_1x04_P2.54mm_Vertical, symbol Connector_Generic:Conn_01x04
- removed IO1, PM2: Conn_01x08_MountingPin, Connector_Molex:Molex_PicoBlade_53261-0871_1x08-1MP_P1.25mm_Horizontal, symbol Connector_Generic_MountingPin:Conn_01x08_MountingPin
- removed S*2: Co2-S8, AG-PRO-Library:Co2-S8, symbol AG-PRO_Library:Co2-S8
- removed U4: LM1117-3.3, Package_TO_SOT_SMD:SOT-223-3_TabPin2, symbol Regulator_Linear:AMS1117-3.3
- added C14: 22uf, Capacitor_SMD:C_0603_1608Metric, symbol Device:C
- added C15, C22, C24: 0.1uf, Capacitor_SMD:C_0603_1608Metric, symbol Device:C
- added C23: 10uf, Capacitor_SMD:C_0603_1608Metric, symbol Device:C
- added J1: BMV080, symbol Connector_Generic:Conn_01x13
- added J2: Conn_01x08, symbol Connector_Generic:Conn_01x08
- added J3: Pogo1, Connector_PinHeader_2.54mm:PinHeader_1x05_P2.54mm_Vertical, symbol Connector_Generic:Conn_01x05
- added J4: Pogo2, Connector_PinHeader_2.54mm:PinHeader_1x05_P2.54mm_Vertical, symbol Connector_Generic:Conn_01x05
- added J5: Pogo3, Connector_PinHeader_2.54mm:PinHeader_1x05_P2.54mm_Vertical, symbol Connector_Generic:Conn_01x05
- added L1: 2.2uH, symbol Device:L
- added R18: 10k, Resistor_SMD:R_0603_1608Metric, symbol Device:R
- added R20: 33.2k, Resistor_SMD:R_0603_1608Metric, symbol Device:R
- added R9: 10k, Resistor_SMD:R_0603_1608Metric, symbol Device:R_Small
- added U1: TPS564201, Package_TO_SOT_SMD:SOT-23-6, symbol Regulator_Switching:TPS56339DDC
- C13: value 0.1uf -> 22uf; LCSC Part # C1590 -> C86295
- C17: value 0.1uf -> 10uf
- C18: value 0.1uf -> 2uf; LCSC Part # C1590 -> C86295
Connections:
- net +3.3V: now also C13.1, C14.1, C22.1, J1.1 (Pin_1), J1.10 (Pin_10), J1.3 (Pin_3), J1.7 (Pin_7), J1.8 (Pin_8), J2.2 (Pin_2), J3.5 (Pin_5), J4.5 (Pin_5), J5.5 (Pin_5), L1.2, R20.2
- net +5V: now also C23.1, C24.1, R18.1, U1.3 (VIN); no longer C13.1
- net GND: now also C14.2, C22.2, C23.2, C24.2, J1.11 (Pin_11), J1.2 (Pin_2), J1.4 (Pin_4), J1.9 (Pin_9), J2.1 (Pin_1), J2.8 (Pin_8), J3.1 (Pin_1), J4.1 (Pin_1), J5.1 (Pin_1), R9.2, U1.1 (GND)
- net IO3: now also J2.7 (Pin_7), J3.4 (Pin_4)
- net IO4: now also J4.4 (Pin_4)
- net IO5: now also J5.4 (Pin_4)
- net RX_1_PMS: now also J3.2 (Pin_2)
- net SCL: now also J1.6 (Pin_6), J2.4 (Pin_4), J4.2 (Pin_2), J5.2 (Pin_2)
- net SDA: now also J1.5 (Pin_5), J2.3 (Pin_3), J4.3 (Pin_3), J5.3 (Pin_3)
- net TX_1_PMS: now also J3.3 (Pin_3)
- net RX_2_PMS renamed IRQ
- net IRQ: now also J1.12 (Pin_12)
- net TX_2_PMS renamed IO1
- net IO1: now also J2.5 (Pin_5)
- new net: C15.1, L1.1, U1.2 (SW)
- new net: C15.2, U1.6 (BOOT)
- new net: R18.2, U1.5 (EN)
- new net: R20.1, R9.1, U1.4 (FB)
- no-connect marks 10 -> 3
Other:
- note added: "BOSCH PMS"
- note removed: "I2C device connectors"
- note removed: "PMS sensor connector"

Commit message: Rev 2.0
Parts:
- J1: footprint (none) -> 503566-1302:5035661302
- J2: footprint (none) -> ZAir:S12
- L1: footprint (none) -> Inductor_SMD:L_0603_1608Metric
- USB1: footprint AG-PRO-Library:918-418K2022Y40000 -> Connector_USB:USB_C_Receptacle_Molex_105450-0101
Changed lines of the file:
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@@
 			)
 		)
-		(property "Footprint" "AG-PRO-Library:918-418K2022Y40000"
+		(property "Footprint" "Connector_USB:USB_C_Receptacle_Molex_105450-0101"
 			(at 51.435 57.785 0)
 			(hide yes)
@@
 			)
 		)
-		(property "Footprint" ""
+		(property "Footprint" "ZAir:S12"
 			(at 111.76 231.14 0)
 			(hide yes)
@@
 			)
 		)
-		(property "Footprint" ""
+		(property "Footprint" "Inductor_SMD:L_0603_1608Metric"
 			(at 186.69 35.56 0)
 			(hide yes)
@@
 			)
 		)
-		(property "Footprint" ""
+		(property "Footprint" "503566-1302:5035661302"
 			(at 349.25 58.42 0)
 			(hide yes)
